Commit message: replaced meshes in <visual> tags with geometry from <collision> tags inside xacro files

File: forklift_description/urdf/forklift.xacro (robot description, xacro)
@@ -39,7 +39,7 @@
     </collision>
     <visual>
-      <origin xyz="-0.89856 0 1.08726" rpy="0 0 ${PI/2}"/> <!-- -0.00203 -0.06282 1.08726-->
+      <origin xyz="-1 0 ${height/2 + 0.2}" rpy="0 0 0"/>
       <geometry>
-	     <mesh filename="package://forklift_description/meshes/forklift_body.dae"/>
+             <box size="${length} ${width} ${height}"/>
       </geometry>
     </visual>

File: forklift_description/urdf/forklift_back_wheels.xacro (robot description, xacro)
@@ -10,7 +10,7 @@
   <link name="forklift_wheelBR">
     <visual>
-      <origin xyz="0 0 0" rpy="0 0 ${PI+PI/2}"/>
+      <origin xyz="0 0 0" rpy="${PI/2} 0 0"/>
       <geometry>
-       <mesh filename="package://forklift_description/meshes/forklift_wheel_back.dae"/>
+       <cylinder radius="${wheelB_radius}" length="${wheelB_width}" />
       </geometry>
     </visual>
@@ -30,7 +30,7 @@
   <link name="forklift_wheelBL">
     <visual>
-      <origin xyz="0 0 0" rpy="0 0 ${PI/2}"/>
+      <origin xyz="0 0 0" rpy="${PI/2} 0 0"/>
       <geometry>
-       <mesh filename="package://forklift_description/meshes/forklift_wheel_back.dae"/>
+       <cylinder radius="${wheelB_radius}" length="${wheelB_width}" />
       </geometry>
     </visual>

File: forklift_description/urdf/forklift_front_wheels.xacro (robot description, xacro)
@@ -16,7 +16,7 @@
     </collision>
     <visual>
-      <origin xyz="0 0 0" rpy="0 0 ${PI+PI/2}"/>
+      <origin xyz="0 0 0" rpy="${PI/2} 0 0"/>
       <geometry>
-       <mesh filename="package://forklift_description/meshes/forklift_wheel_front.dae"/>
+       <cylinder radius="${wheelF_radius}" length="${wheelF_width}" />
       </geometry>
     </visual>
@@ -42,7 +42,7 @@
     </collision>
     <visual>
-      <origin xyz="0 0 0" rpy="0 0 ${PI/2}"/>
+      <origin xyz="0 0 0" rpy="${PI/2} 0 0"/>
       <geometry>
-       <mesh filename="package://forklift_description/meshes/forklift_wheel_front.dae"/>
+       <cylinder radius="${wheelF_radius}" length="${wheelF_width}" />
       </geometry>
     </visual>

File: forklift_description/urdf/forklift_lift.xacro (robot description, xacro)
@@ -27,7 +27,19 @@
     </collision>
     <visual>
-      <origin xyz="-0.89856 0 0" rpy="0 0 ${PI/2}"/>
+      <origin xyz="0.55 0 0.695" rpy="0 0 0"/>
       <geometry>
-       <mesh filename="package://forklift_description/meshes/forklift_lift1.dae"/>
+       <box size="0.1 1.2 1.25"/>
+      </geometry>
+    </visual>
+    <visual>
+      <origin xyz="1.2 0.32 0.06" rpy="0 0 0"/>
+      <geometry>
+       <box size="1.2 0.13 0.03"/>
+      </geometry>
+    </visual>
+    <visual>
+      <origin xyz="1.2 -0.32 0.06" rpy="0 0 0"/>
+      <geometry>
+       <box size="1.2 0.13 0.03"/>
       </geometry>
     </visual>
@@ -53,7 +65,7 @@
     </collision>
     <visual>
-      <origin xyz="-0.89856 0 0" rpy="0 0 ${PI/2}"/>
+      <origin xyz="0.25 0 1.05" rpy="0 0 0"/>
       <geometry>
-       <mesh filename="package://forklift_description/meshes/forklift_lift2.dae"/>
+       <box size="0.3 0.7 2"/>
       </geometry>
     </visual>
